File: stm32-devboard.kicad_pcb (KiCad board)
At the start: 2 copper layers, 15 parts, among them U1 STM32G473CCUx, Y1 Crystal, Y2 Crystal

Commit message: finished preliminary design
Parts:
- added C11: 22uF, Capacitor_SMD:C_0805_2012Metric, F.Cu at (118.3, 55.4)
- added C12: 10uF, Capacitor_SMD:C_0402_1005Metric, F.Cu at (126.9, 61.2)
- added J1: Conn_01x03_Pin, Connector_PinHeader_2.54mm:PinHeader_1x03_P2.54mm_Vertical, F.Cu at (132.6, 64.5)
- added J2: Conn_01x20_Pin, Connector_PinHeader_2.54mm:PinHeader_1x20_P2.54mm_Vertical, F.Cu at (137.2, 54.4)
- added J3: Conn_01x20_Pin, Connector_PinHeader_2.54mm:PinHeader_1x20_P2.54mm_Vertical, F.Cu at (114.3, 54.4)
- added U2: AZ1117-3.3, Package_TO_SOT_SMD:SOT-223-3_TabPin2, F.Cu at (122.9, 57.9)
- moved C9 10.2 mm to (116.8, 78.4), turned to -90 degrees
- moved Y2 8.16 mm to (119.4, 76.7), turned to -90 degrees
- moved C8 7.77 mm to (116.8, 75.7), turned to -90 degrees
- moved C1 7.05 mm to (132.1, 73.4)
- moved C2 7.04 mm to (129.5, 81.3)
- moved C6 6.73 mm to (118.4, 70.4)
- moved C3 6.72 mm to (128.0, 81.3)
- moved C4 6.70 mm to (127.0, 81.3)
- moved Y1 6.68 mm to (119.4, 72.2)
- moved U1 6.65 mm to (126.6, 75.7)
- moved C10 6.64 mm to (122.9, 70.1)
- moved JP1 6.62 mm to (124.9, 67.2)
- moved R1 6.62 mm to (124.9, 70.1)
- moved C5 6.62 mm to (121.9, 70.1)
- moved C7 6.57 mm to (120.4, 70.4)
Connections:
- U1 pad 10: unconnected-(U1-PA2-Pad10) -> /PA2
- U1 pad 11: unconnected-(U1-PA3-Pad11) -> /PA3
- U1 pad 12: unconnected-(U1-PA4-Pad12) -> /PA4
- U1 pad 13: unconnected-(U1-PA5-Pad13) -> /PA5
- U1 pad 14: unconnected-(U1-PA6-Pad14) -> /PA6
- U1 pad 15: unconnected-(U1-PA7-Pad15) -> /PA7
- U1 pad 16: unconnected-(U1-PC4-Pad16) -> /PC4
- U1 pad 17: unconnected-(U1-PB0-Pad17) -> /PB0
- U1 pad 18: unconnected-(U1-PB1-Pad18) -> /PB1
- U1 pad 19: unconnected-(U1-PB2-Pad19) -> /PB2
- U1 pad 2: unconnected-(U1-PC13-Pad2) -> /PC13
- U1 pad 22: unconnected-(U1-PB10-Pad22) -> /PB10
- U1 pad 24: unconnected-(U1-PB11-Pad24) -> /PB11
- U1 pad 25: unconnected-(U1-PB12-Pad25) -> /PB12
- U1 pad 26: unconnected-(U1-PB13-Pad26) -> /PB13
- U1 pad 27: unconnected-(U1-PB14-Pad27) -> /PB14
- U1 pad 28: unconnected-(U1-PB15-Pad28) -> /PB15
- U1 pad 29: unconnected-(U1-PC6-Pad29) -> /PC6
- U1 pad 30: unconnected-(U1-PA8-Pad30) -> /PA8
- U1 pad 31: unconnected-(U1-PA9-Pad31) -> /PA9
- U1 pad 32: unconnected-(U1-PA10-Pad32) -> /PA10
- U1 pad 33: unconnected-(U1-PA11-Pad33) -> /PA11
- U1 pad 34: unconnected-(U1-PA12-Pad34) -> /PA12
- U1 pad 39: unconnected-(U1-PC10-Pad39) -> /PC10
- U1 pad 40: unconnected-(U1-PC11-Pad40) -> /PC11
- U1 pad 41: unconnected-(U1-PB3-Pad41) -> /PB3
- U1 pad 42: unconnected-(U1-PB4-Pad42) -> /PB4
- U1 pad 43: unconnected-(U1-PB5-Pad43) -> /PB5
- U1 pad 44: unconnected-(U1-PB6-Pad44) -> /PB6
- U1 pad 45: unconnected-(U1-PB7-Pad45) -> /PB7
- U1 pad 47: unconnected-(U1-PB9-Pad47) -> /PB9
- U1 pad 8: unconnected-(U1-PA0-Pad8) -> /PA0
- U1 pad 9: unconnected-(U1-PA1-Pad9) -> /PA1
Routing:
- net +3.3V: track 4.57 -> 75.4 mm, vias 1 -> 6
- net /PB5: track 0.00 -> 26.7 mm
- net /PB2: track 0.00 -> 26.1 mm
- net /PB6: track 0.00 -> 24.0 mm
- net /PB1: track 0.00 -> 23.4 mm
- net /PB10: track 0.00 -> 22.1 mm
- net /PB7: track 0.00 -> 21.3 mm
- net /PB4: track 0.00 -> 21.1 mm
- net /PB0: track 0.00 -> 20.7 mm
- net /PB11: track 0.00 -> 19.7 mm
- net /PB3: track 0.00 -> 19.6 mm
- net /PC4: track 0.00 -> 17.9 mm
- net /PC10: track 0.00 -> 17.7 mm
- net /PB12: track 0.00 -> 17.7 mm
- net /PC11: track 0.00 -> 17.4 mm
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- added copper zone on F.Cu, net +3.3V
- added copper zone on B.Cu, net GND
- added copper zone on F.Cu, net GND
Other:
- board outline added: 25.9 x 51.3 mm
- board text added: "1"
- board text added: "10"
- board text added: "11"
- board text added: "12"
- board text added: "13"
- board text added: "14"
- board text added: "15"
- board text added: "16"
- board text added: "17"
- board text added: "18"
- board text added: "19"
- board text added: "2"
- board text added: "20"
- board text added: "21"
- board text added: "22"
- board text added: "23"
- board text added: "24"
- board text added: "25"
- board text added: "26"
- board text added: "27"
- board text added: "28"
- board text added: "29"
- board text added: "3"
- board text added: "30"
- board text added: "31"
- board text added: "32"
- board text added: "33"
- board text added: "34"
- board text added: "35"
- board text added: "36"
- board text added: "37"
- board text added: "38"
- board text added: "39"
- board text added: "4"
- board text added: "40"
- board text added: "5"
- board text added: "6"
- board text added: "7"
- board text added: "8"
- board text added: "9"

Commit message: final revision
Parts:
- removed the Y2 at (119.4, 76.7)
- added C1: 100n, Capacitor_SMD:C_0402_1005Metric, F.Cu at (128.0, 59.2)
- added R2: 220, Resistor_SMD:R_0402_1005Metric, F.Cu at (119.1, 78.7)
- added Y1: X322524MSB4SI, Crystal:Crystal_SMD_3225-4Pin_3.2x2.5mm, F.Cu at (118.1, 75.9)
- C10: renamed from C7; value 5p -> 4p
- C6: renamed from C8; value 24p -> 30p
- C7: renamed from C9; value 24p -> 30p
- C9: renamed from C6; value 5p -> 4p
- J1: value Conn_01x03_Pin -> Conn_01x04_Pin; footprint Connector_PinHeader_2.54mm:PinHeader_1x03_P2.54mm_Vertical -> Connector_PinHeader_2.54mm:PinHeader_1x04_P2.54mm_Vertical
- Y2: renamed from Y1; value Crystal -> X161032768KJD2SI; footprint Crystal:Crystal_SMD_G8-2Pin_3.2x1.5mm -> Crystal:Crystal_SMD_MicroCrystal_CM9V-T1A-2Pin_1.6x1.0mm
- moved C6 2.55 mm to (117.1, 73.2), turned to 180 degrees
- moved J1 2.54 mm to (132.6, 62.0)
- moved C7 0.46 mm to (117.1, 78.7), turned to 180 degrees
- renumbered C10 to C12, C12 to C13, C1 to C2, C2 to C3, C3 to C4, C4 to C5, C5 to C8
Connections:
- C7 pad 1: /OSC_OUT -> Net-(C7-Pad1)
- J1 pad 1: /TDI -> /NRST
- J1 pad 2: /SWCLK -> /TDI
- J1 pad 3: /SWDIO -> /SWCLK
Routing:
- net /NRST: track 3.13 -> 35.4 mm, vias 1 -> 2
- net /PC10: track 17.7 -> 21.5 mm
- net /OSC_OUT: track 8.90 -> 5.87 mm
- net Net-(C7-Pad1): track 0.00 -> 2.88 mm
- net /PC11: track 17.4 -> 20.1 mm
- net /OSC_IN: track 6.71 -> 8.68 mm
- net GND: track 8.81 -> 9.91 mm, vias 18 -> 17
- net /PB4: track 21.1 -> 21.8 mm
- net /PB3: track 19.6 -> 20.2 mm
- net +3.3V: track 75.4 -> 76.0 mm
Other:
- board text removed: "10"
- board text removed: "9"
