File: stm32-devboard.kicad_sch (KiCad schematic)
At the start: 16 parts, among them J1 Conn_01x20_Pin, U1 STM32G473CCUx, Y1 Crystal, Y2 Crystal

Commit message: finished preliminary design
Parts:
- added C11: 22uF, Capacitor_SMD:C_0805_2012Metric, symbol Device:C_Small
- added C12: 10uF, Capacitor_SMD:C_0402_1005Metric, symbol Device:C_Small
- added J1: Conn_01x03_Pin, Connector_PinHeader_2.54mm:PinHeader_1x03_P2.54mm_Vertical, symbol Connector:Conn_01x03_Pin
- added J2: Conn_01x20_Pin, Connector_PinHeader_2.54mm:PinHeader_1x20_P2.54mm_Vertical, symbol Connector:Conn_01x20_Pin
- added U2: AZ1117-3.3, Package_TO_SOT_SMD:SOT-223-3_TabPin2, symbol Regulator_Linear:AZ1117-3.3
- J3: renamed from J1; footprint (none) -> Connector_PinHeader_2.54mm:PinHeader_1x20_P2.54mm_Vertical
- Y1: footprint Crystal:Crystal_SMD_G8-2Pin_3.2x1.5mm -> Crystal:Crystal_SMD_MicroCrystal_CM9V-T1A-2Pin_1.6x1.0mm
Connections:
- net +3.3V: now also C12.1, J2.1 (Pin_1), U2.2 (VO)
- net GND: now also J3.20 (Pin_20), J3.6 (Pin_6), C11.2, C12.2, J2.19 (Pin_19), J2.20 (Pin_20), J2.6 (Pin_6), U2.1 (GND)
- net PA0: now also J3.8 (Pin_8)
- net PA1: now also J3.9 (Pin_9)
- net PA10: now also J2.9 (Pin_9)
- net PA11: now also J2.8 (Pin_8)
- net PA12: now also J2.7 (Pin_7)
- net PA2: now also J3.10 (Pin_10)
- net PA3: now also J3.11 (Pin_11)
- net PA4: now also J3.12 (Pin_12)
- net PA5: now also J3.13 (Pin_13)
- net PA6: now also J3.14 (Pin_14)
- net PA7: now also J3.15 (Pin_15)
- net PA8: now also J2.11 (Pin_11)
- net PA9: now also J2.10 (Pin_10)
- net PB0: now also J3.17 (Pin_17)
- net PB1: now also J3.18 (Pin_18)
- net PB10: now also J2.18 (Pin_18)
- net PB11: now also J2.17 (Pin_17)
- net PB12: now also J2.16 (Pin_16)
- net PB13: now also J2.15 (Pin_15)
- net PB14: now also J2.14 (Pin_14)
- net PB15: now also J2.13 (Pin_13)
- net PB2: now also J3.19 (Pin_19)
- net PB3: now also J2.3 (Pin_3)
- net PB4: now also J2.2 (Pin_2)
- net PB5: now also J3.2 (Pin_2)
- net PB6: now also J3.3 (Pin_3)
- net PB7: now also J3.4 (Pin_4)
- net PB9: now also J3.5 (Pin_5)
- net PC10: now also J2.5 (Pin_5)
- net PC11: now also J2.4 (Pin_4)
- net PC13: now also J3.7 (Pin_7)
- net PC4: now also J3.16 (Pin_16)
- net PC6: now also J2.12 (Pin_12)
- net SWCLK: now also J1.2 (Pin_2)
- net SWDIO: now also J1.3 (Pin_3)
- net TDI: now also J1.1 (Pin_1)
- net VBUS: now reaches J3.1 (Pin_1)
- net VBUS: now also C11.1, U2.3 (VI)
Other:
- note added: "Application note for STM32G4 series hardware development"
- note removed: "STM32G473"
- moved on the sheet: J3

Commit message: final revision
Parts:
- removed J1: Conn_01x03_Pin, Connector_PinHeader_2.54mm:PinHeader_1x03_P2.54mm_Vertical, symbol Connector:Conn_01x03_Pin
- removed Y2: Crystal, Crystal:Crystal_SMD_Abracon_ABM3-2Pin_5.0x3.2mm, symbol Device:Crystal
- added C1: 100n, Capacitor_SMD:C_0402_1005Metric, symbol Device:C_Small
- added J1: Conn_01x04_Pin, Connector_PinHeader_2.54mm:PinHeader_1x04_P2.54mm_Vertical, symbol Connector:Conn_01x04_Pin
- added R2: 220, Resistor_SMD:R_0402_1005Metric, symbol Device:R_Small
- added Y1: X322524MSB4SI, Crystal:Crystal_SMD_3225-4Pin_3.2x2.5mm, symbol Device:Crystal_GND24_Small
- C10: renamed from C7; value 5p -> 4p
- C6: renamed from C8; value 24p -> 30p
- C7: renamed from C9; value 24p -> 30p
- C9: renamed from C6; value 5p -> 4p
- Y2: renamed from Y1; value Crystal -> X161032768KJD2SI
- renumbered C10 to C12, C12 to C13, C1 to C2, C2 to C3, C3 to C4, C4 to C5, C5 to C8
Connections:
- net GND: now also C1.2, Y1.2, Y1.4
- net NRST: now also C1.1, J1.1 (Pin_1)
- net OSC_IN: now also Y1.3
- net OSC_OUT: now also R2.2; no longer C7.1
- net SWCLK: now also J1.3 (Pin_3)
- net SWDIO: now also J1.4 (Pin_4)
- net TDI: now also J1.2 (Pin_2)
- new net: C7.1, R2.1, Y1.1
Other:
- moved on the sheet: C11, C13, C6, C7, U2
